File: hardware/68008.brd (EAGLE design)
At the start: 151.4 x 117.5 mm, 41 parts, among them IC1 74HCT139N, IC10 74HCT00N, IC2 74LS373N, IC3 74HCT245DW, IC4 74HCT245DW, IC5 74HCT00N, IC6 74HCT139N, IC7 DS1813, IC9 74HCT138N

Commit message: PCB updated
Parts:
- removed U$2, U$4: 62256, memory-sram:DIL28-6
- added U1, U2: AS6C4008-55PCN, Alliance_Memory_By_element14_Batch_1:DIP254P1524X393-32
- R9: device rcl:0204/7 -> rcl:R1206
- moved C12 33.0 mm to (95.9, 18.7)
- moved IC6 32.9 mm to (92.1, 6.67)
- moved C17 32.4 mm to (82.2, 18.7)
- moved IC1 32.3 mm to (78.4, 6.67)
- moved C11 28.7 mm to (65.4, 18.7)
- moved IC5 28.6 mm to (61.6, 7.94)
- moved R9 22.9 mm to (106.8, 10.5), flipped to the bottom
- moved C13 16.5 mm to (111.4, 18.7)
- moved IC9 16.5 mm to (107.6, 6.67)
- moved C1 4.45 mm to (43.2, 37.3)
- moved C2 4.45 mm to (63.5, 37.3)
- moved U$1 4.44 mm to (15.2, 50.2)
- moved C3 4.44 mm to (83.8, 37.3)
Connections:
- removed net BANK_A13: IC2.2, U$2.26
- removed net BANK_A14: IC2.5, U$2.1
- removed net CS_RAM32K: IC1.4, U$4.20
- new net BANK_A17: IC2.2, U2.30
- new net BANK_A18: IC2.5, U2.1
- new net CLK: U$1.34
- new net CS_RAM512K: IC1.4, U1.22
- net A0: now also U1.12, U2.12; no longer U$2.10, U$4.10
- net A1: now also U1.11, U2.11; no longer U$2.9, U$4.9
- net A10: now also U1.23, U2.23; no longer IC9.1, U$2.21, U$4.21
- net A11: now also U1.25, U2.25; no longer IC9.2, U$2.23, U$4.23
- net A12: now also U1.4, U2.4; no longer IC9.3, U$2.2, U$4.2
- net A13: now also U1.28, U2.28; no longer IC6.14, U$4.26
- net A14: now also IC9.1, U1.3, U2.3; no longer IC6.2, U$4.1
- net A15: now also IC9.2, U1.31, U2.31; no longer IC1.2
- net A16: now also IC9.3, U1.2, U2.2
- net A17: now also IC6.14, U1.30
- net A18: now also IC6.2, U1.1
- net A19: now also IC1.2
- net A2: now also U1.10, U2.10; no longer U$2.8, U$4.8
- net A3: now also U1.9, U2.9; no longer U$2.7, U$4.7
- net A4: now also U1.8, U2.8; no longer U$2.6, U$4.6
- net A5: now also U1.7, U2.7; no longer U$2.5, U$4.5
- net A6: now also U1.6, U2.6; no longer U$2.4, U$4.4
- net A7: now also U1.5, U2.5; no longer U$2.3, U$4.3
- net A8: now also U1.27, U2.27; no longer U$2.25, U$4.25
- net A9: now also U1.26, U2.26; no longer U$2.24, U$4.24
- net CS_BANKED_RAM: now also U2.22; no longer U$2.20
- net D0: now also U1.13, U2.13; no longer U$2.11, U$4.11
- net D1: now also U1.14, U2.14; no longer U$2.12, U$4.12
- net D2: now also U1.15, U2.15; no longer U$2.13, U$4.13
- net D3: now also U1.17, U2.17; no longer U$2.15, U$4.15
- net D4: now also U1.18, U2.18; no longer U$2.16, U$4.16
- net D5: now also U1.19, U2.19; no longer U$2.17, U$4.17
- net D6: now also U1.20, U2.20; no longer U$2.18, U$4.18
- net D7: now also U1.21, U2.21; no longer U$2.19, U$4.19
- net GND: now also U$1.15, U$1.35, U1.16, U2.16; no longer U$2.14, U$4.14
- net RD: now also U1.24, U2.24; no longer U$2.22, U$4.22
- net RW: now also U$1.30
- net VCC: now also U1.32, U2.32; no longer U$2.28, U$4.28
- net WR: now also U1.29, U2.29; no longer U$2.27, U$4.27
Routing:
- net A18: track 0.00 -> 131.3 mm, vias 0 -> 4
- net CS_RAM512K: track 0.00 -> 93.3 mm, vias 0 -> 2
- net A2: track 75.7 -> 152.4 mm, vias 0 -> 2
- net A16: track 0.00 -> 71.4 mm, vias 0 -> 2
- net A3: track 76.2 -> 146.1 mm, vias 0 -> 2
- net CS_RAM32K: track 59.3 -> 0.00 mm, vias 2 -> 0
- net BANK_A17: track 0.00 -> 57.5 mm, vias 0 -> 2
- net BANK_A18: track 0.00 -> 56.7 mm, vias 0 -> 2
- net A7: track 85.5 -> 142.1 mm, vias 2 -> 4
- net A4: track 76.8 -> 131.4 mm, vias 0 -> 2
- net A17: track 0.00 -> 53.8 mm, vias 0 -> 3
- net BANK_A13: track 52.6 -> 0.00 mm, vias 2 -> 0
- net BANK_A14: track 52.3 -> 0.00 mm, vias 2 -> 0
- net A5: track 77.9 -> 126.8 mm, vias 0 -> 2
- net A6: track 79.7 -> 124.1 mm, vias 2 -> 4
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Other:
- board size 151.4 x 117.5 mm -> 151.4 x 124.5 mm
- board text added: "MC68008 CPU BOARD"
- board text removed: "MC6802 CPU BOARD"
