File: hardware/68008.sch (EAGLE design)
At the start: 41 parts, among them IC1 74HCT139N, IC10 74HCT00N, IC2 74LS373N, IC3 74HCT245DW, IC4 74HCT245DW, IC5 74HCT00N, IC6 74HCT139N, IC7 DS1813, IC9 74HCT138N

Commit message: PCB updated
Parts:
- removed U$2, U$4: 62256, memory-sram:62256
- added U1, U2: AS6C4008-55PCN, Alliance_Memory_By_element14_Batch_1:AS6C4008-55PCN
- R9: device rcl:R-EU_0204/7 -> rcl:R-EU_R1206
Connections:
- removed net BANK_A13: IC2A.1Q, U$2.A13
- removed net BANK_A14: IC2A.2Q, U$2.A14
- removed net CS_RAM32K: IC1A.Y0, U$4.!CS
- new net BANK_A17: IC2A.1Q, U2.A17
- new net BANK_A18: IC2A.2Q, U2.A18
- new net CLK: U$1.CLK
- new net CS_RAM512K: IC1A.Y0, U1.CE
- net A0: now also U1.A0, U2.A0; no longer U$2.A0, U$4.A0
- net A1: now also U1.A1, U2.A1; no longer U$2.A1, U$4.A1
- net A10: now also U1.A10, U2.A10; no longer IC9A.A, U$2.A10, U$4.A10
- net A11: now also U1.A11, U2.A11; no longer IC9A.B, U$2.A11, U$4.A11
- net A12: now also U1.A12, U2.A12; no longer IC9A.C, U$2.A12, U$4.A12
- net A13: now also U1.A13, U2.A13; no longer IC6B.A, U$4.A13
- net A14: now also IC9A.A, U1.A14, U2.A14; no longer IC6A.A, U$4.A14
- net A15: now also IC9A.B, U1.A15, U2.A15; no longer IC1A.A
- net A16: now also IC9A.C, U1.A16, U2.A16
- net A17: now also IC6B.A, U1.A17
- net A18: now also IC6A.A, U1.A18
- net A19: now also IC1A.A
- net A2: now also U1.A2, U2.A2; no longer U$2.A2, U$4.A2
- net A3: now also U1.A3, U2.A3; no longer U$2.A3, U$4.A3
- net A4: now also U1.A4, U2.A4; no longer U$2.A4, U$4.A4
- net A5: now also U1.A5, U2.A5; no longer U$2.A5, U$4.A5
- net A6: now also U1.A6, U2.A6; no longer U$2.A6, U$4.A6
- net A7: now also U1.A7, U2.A7; no longer U$2.A7, U$4.A7
- net A8: now also U1.A8, U2.A8; no longer U$2.A8, U$4.A8
- net A9: now also U1.A9, U2.A9; no longer U$2.A9, U$4.A9
- net CS_BANKED_RAM: now also U2.CE; no longer U$2.!CS
- net D0: now also U1.DQ0, U2.DQ0; no longer U$2.D0, U$4.D0
- net D1: now also U1.DQ1, U2.DQ1; no longer U$2.D1, U$4.D1
- net D2: now also U1.DQ2, U2.DQ2; no longer U$2.D2, U$4.D2
- net D3: now also U1.DQ3, U2.DQ3; no longer U$2.D3, U$4.D3
- net D4: now also U1.DQ4, U2.DQ4; no longer U$2.D4, U$4.D4
- net D5: now also U1.DQ5, U2.DQ5; no longer U$2.D5, U$4.D5
- net D6: now also U1.DQ6, U2.DQ6; no longer U$2.D6, U$4.D6
- net D7: now also U1.DQ7, U2.DQ7; no longer U$2.D7, U$4.D7
- net GND: now also U$1.GND@1, U$1.GND@2, U1.VSS, U2.VSS; no longer U$2.VSS, U$4.VSS
- net RD: now also U1.OE, U2.OE; no longer U$2.!OE, U$4.!OE
- net RW: now also U$1.R/!W
- net VCC: now also U1.VCC, U2.VCC; no longer U$2.VCC, U$4.VCC
- net WR: now also U1.WE, U2.WE; no longer U$2.!WE, U$4.!WE
